File: led-ring.kicad_pcb (KiCad board)
At the start: 2 copper layers, 48 x 70 mm, 13 parts, among them U1 USB-C-6-PIN, U2 USB-C-6-PIN, U3 AMS1117-3.3

Commit message: 。
Parts:
- added SW1: DP3T, switch:SS-1400S-L1, F.Cu at (8.38, 35.8)
- moved C1 15.1 mm to (5.74, 25.1)
- moved C2 15.1 mm to (5.84, 22.5)
- moved U1 11.7 mm to (-4.47, 28.5)
- moved U2 7.00 mm to (-4.47, 35.0)
- moved D7 3.11 mm to (-14.8, 14.8), turned to 225 degrees
- moved D3 2.43 mm to (14.8, -14.8), turned to 45 degrees
- moved D6 0.91 mm to (-21.0, 0.00), turned to 180 degrees
- moved D4 0.89 mm to (0.00, -21.0), turned to 90 degrees
- moved D5 0.80 mm to (-14.8, -14.8), turned to 135 degrees
- moved D2 0.67 mm to (21.0, 0.00)
- moved D1 0.64 mm to (14.8, 14.8), turned to 315 degrees
- moved D8 0.31 mm to (0.00, 21.0), turned to 270 degrees
Connections:
- C1 pad 1: VBUS -> VBUS3
- U1 pad 2: VBUS -> VBUS1
- U1 pad 3: Net-(U1-Pad3) -> (no net)
- U1 pad 4: Net-(U1-Pad4) -> (no net)
- U1 pad 5: VBUS -> VBUS1
- U2 pad 2: VBUS -> VBUS2
- U2 pad 3: Net-(U2-Pad3) -> (no net)
- U2 pad 4: Net-(U2-Pad4) -> (no net)
- U2 pad 5: VBUS -> VBUS2
- U3 pad 3: VBUS -> VBUS3
Routing:
- added copper zone on F.Cu, net +3V3
- added copper zone on B.Cu, net GND
Other:
- rule via_min_drill: 0.3 -> 0.254

Commit message: .
Parts:
- moved C2 18.8 mm to (-12.4, 18.0), turned to 45 degrees
- moved U2 6.95 mm to (-4.47, 28.0)
- moved U1 6.55 mm to (-4.47, 35.0)
- moved C1 0.30 mm to (5.59, 24.9), turned to 90 degrees
Routing:
- net VBUS3: track 0.00 -> 24.8 mm
- net VBUS2: track 0.00 -> 15.8 mm
- net VBUS1: track 0.00 -> 14.9 mm
- net GND: track 0.00 -> 1.79 mm, vias 0 -> 19
Changed lines of the file:
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@@
     (thickness 1.6)
     (drawings 7)
-    (tracks 0)
+    (tracks 46)
     (zones 0)
     (modules 14)
@@
   (setup
     (last_trace_width 0.25)
+    (user_trace_width 0.5)
     (trace_clearance 0.2)
     (zone_clearance 0.508)
@@
   )
   (module Connector_Custom:TYPE-C-31-D-01 (layer B.Cu)
-    (at -4.467 34.953)
+    (at -4.467 28)
     (fp_text reference U2 (at 0 -3.675) (layer B.SilkS)
       (effects (font (size 1 1) (thickness 0.15)) (justify mirror))
@@
   )
   (module Connector_Custom:TYPE-C-31-D-01 (layer B.Cu)
-    (at -4.467 28.453)
+    (at -4.467 35)
     (fp_text reference U1 (at 0 -3.675) (layer B.SilkS)
       (effects (font (size 1 1) (thickness 0.15)) (justify mirror))
@@
   )
   (module Capacitor_SMD:C_0402_1005Metric (layer F.Cu)
-    (at 5.842 22.479)
+    (at -12.446 18.034 45)
     (descr "Capacitor SMD 0402 (1005 Metric), square (rectangular) end terminal, IPC_7351 nominal, (Body size source: IPC-SM-782 page 76, https://www.pcb-3d.com/wordpress/wp-content/uploads/ipc-sm-782a_amendment_1_and_2.pdf), generated with kicad-footprint-generator")
     (tags capacitor)
     (attr smd)
-    (fp_text reference C2 (at 0 -1.16) (layer F.SilkS)
-      (effects (font (size 1 1) (thickness 0.15)))
-    )
-    (fp_text value 10uF (at 0 1.16) (layer F.Fab)
+    (fp_text reference C2 (at 0 -1.16 45) (layer F.SilkS)
+      (effects (font (size 1 1) (thickness 0.15)))
+    )
+    (fp_text value 10uF (at -0.762 -0.762 45) (layer F.Fab) hide
       (effects (font (size 1 1) (thickness 0.15)))
     )
@@
     (fp_line (start 0.91 -0.46) (end 0.91 0.46) (layer F.CrtYd) (width 0.05))
     (fp_line (start 0.91 0.46) (end -0.91 0.46) (layer F.CrtYd) (width 0.05))
-    (fp_text user %R (at 0 0) (layer F.Fab)
+    (fp_text user %R (at 0 0 45) (layer F.Fab)
       (effects (font (size 0.25 0.25) (thickness 0.04)))
     )
-    (pad 2 smd roundrect (at 0.48 0) (size 0.56 0.62) (layers F.Cu F.Paste F.Mask) (roundrect_rratio 0.25)
-      (net 1 GND))
-    (pad 1 smd roundrect (at -0.48 0) (size 0.56 0.62) (layers F.Cu F.Paste F.Mask) (roundrect_rratio 0.25)
+    (pad 2 smd roundrect (at 0.48 0 45) (size 0.56 0.62) (layers F.Cu F.Paste F.Mask) (roundrect_rratio 0.25)
+      (net 1 GND))
+    (pad 1 smd roundrect (at -0.48 0 45) (size 0.56 0.62) (layers F.Cu F.Paste F.Mask) (roundrect_rratio 0.25)
       (net 2 +3V3))
     (model ${KISYS3DMOD}/Capacitor_SMD.3dshapes/C_0402_1005Metric.wrl
@@
   )
   (module Capacitor_SMD:C_0402_1005Metric (layer F.Cu)
-    (at 5.743 25.146)
+    (at 5.588 24.892 90)
     (descr "Capacitor SMD 0402 (1005 Metric), square (rectangular) end terminal, IPC_7351 nominal, (Body size source: IPC-SM-782 page 76, https://www.pcb-3d.com/wordpress/wp-content/uploads/ipc-sm-782a_amendment_1_and_2.pdf), generated with kicad-footprint-generator")
     (tags capacitor)
     (attr smd)
-    (fp_text reference C1 (at 0 -1.16) (layer F.SilkS)
-      (effects (font (size 1 1) (thickness 0.15)))
-    )
-    (fp_text value 10uF (at 0 1.16) (layer F.Fab)
+    (fp_text reference C1 (at 0 -1.16 90) (layer F.SilkS)
+      (effects (font (size 1 1) (thickness 0.15)))
+    )
+    (fp_text value 10uF (at 0 1.16 90) (layer F.Fab)
       (effects (font (size 1 1) (thickness 0.15)))
     )
@@
     (fp_line (start 0.91 -0.46) (end 0.91 0.46) (layer F.CrtYd) (width 0.05))
     (fp_line (start 0.91 0.46) (end -0.91 0.46) (layer F.CrtYd) (width 0.05))
-    (fp_text user %R (at 0 0) (layer F.Fab)
+    (fp_text user %R (at 0 0 90) (layer F.Fab)
       (effects (font (size 0.25 0.25) (thickness 0.04)))
     )
-    (pad 2 smd roundrect (at 0.48 0) (size 0.56 0.62) (layers F.Cu F.Paste F.Mask) (roundrect_rratio 0.25)
-      (net 1 GND))
-    (pad 1 smd roundrect (at -0.48 0) (size 0.56 0.62) (layers F.Cu F.Paste F.Mask) (roundrect_rratio 0.25)
+    (pad 2 smd roundrect (at 0.48 0 90) (size 0.56 0.62) (layers F.Cu F.Paste F.Mask) (roundrect_rratio 0.25)
+      (net 1 GND))
+    (pad 1 smd roundrect (at -0.48 0 90) (size 0.56 0.62) (layers F.Cu F.Paste F.Mask) (roundrect_rratio 0.25)
       (net 3 VBUS3))
     (model ${KISYS3DMOD}/Capacitor_SMD.3dshapes/C_0402_1005Metric.wrl
@@
   (gr_line (start -12 20.78461) (end -12 41) (layer Edge.Cuts) (width 0.05))
   (gr_arc (start 0 0) (end -12 20.78461) (angle 300) (layer Edge.Cuts) (width 0.05))
+  (via (at 0.635 19.812) (size 0.508) (drill 0.254) (layers F.Cu B.Cu) (net 1))
+  (via (at -0.508 20.447) (size 0.508) (drill 0.254) (layers F.Cu B.Cu) (net 1))
+  (via (at 14.986 14.224) (size 0.508) (drill 0.254) (layers F.Cu B.Cu) (net 1))
+  (via (at 13.335 14.224) (size 0.508) (drill 0.254) (layers F.Cu B.Cu) (net 1))
+  (via (at 20.574 0.508) (size 0.508) (drill 0.254) (layers F.Cu B.Cu) (net 1))
+  (via (at 19.558 -0.381) (size 0.508) (drill 0.254) (layers F.Cu B.Cu) (net 1))
+  (via (at 14.859 -14.224) (size 0.508) (drill 0.254) (layers F.Cu B.Cu) (net 1))
+  (via (at 13.716 -14.224) (size 0.508) (drill 0.254) (layers F.Cu B.Cu) (net 1))
+  (via (at 0.508 -19.558) (size 0.508) (drill 0.254) (layers F.Cu B.Cu) (net 1))
+  (via (at -0.508 -20.574) (size 0.508) (drill 0.254) (layers F.Cu B.Cu) (net 1))
+  (via (at -13.589 -14.097) (size 0.508) (drill 0.254) (layers F.Cu B.Cu) (net 1))
+  (via (at -14.859 -14.224) (size 0.508) (drill 0.254) (layers F.Cu B.Cu) (net 1))
+  (via (at -19.685 -0.381) (size 0.508) (drill 0.254) (layers F.Cu B.Cu) (net 1))
+  (via (at -20.447 0.508) (size 0.508) (drill 0.254) (layers F.Cu B.Cu) (net 1))
+  (via (at -13.589 14.224) (size 0.508) (drill 0.254) (layers F.Cu B.Cu) (net 1))
+  (via (at -14.859 14.224) (size 0.508) (drill 0.254) (layers F.Cu B.Cu) (net 1))
+  (via (at -11.684 17.272) (size 0.508) (drill 0.254) (layers F.Cu B.Cu) (net 1))
+  (segment (start -12.106589 17.694589) (end -11.684 17.272) (width 0.25) (layer F.Cu) (net 1))
+  (segment (start -9.778 18.416) (end -9.779 18.415) (width 0.25) (layer F.Cu) (net 1))
+  (via (at -9.779 18.415) (size 0.508) (drill 0.254) (layers F.Cu B.Cu) (net 1))
+  (segment (start -9.778 19.074) (end -9.778 18.416) (width 0.25) (layer F.Cu) (net 1))
+  (via (at 5.588 23.876) (size 0.508) (drill 0.254) (layers F.Cu B.Cu) (net 1))
+  (segment (start 5.588 24.412) (end 5.588 23.876) (width 0.25) (layer F.Cu) (net 1))
+  (segment (start 5.632 27.222) (end 5.632 31.814) (width 0.5) (layer F.Cu) (net 3))
+  (segment (start 5.632 25.416) (end 5.588 25.372) (width 0.5) (layer F.Cu) (net 3))
+  (segment (start 5.632 27.222) (end 5.632 25.416) (width 0.5) (layer F.Cu) (net 3))
+  (segment (start 2.921 24.511) (end 5.632 27.222) (width 0.5) (layer F.Cu) (net 3))
+  (segment (start -8.636 24.511) (end 2.921 24.511) (width 0.5) (layer F.Cu) (net 3))
+  (segment (start -9.778 23.369) (end -8.636 24.511) (width 0.5) (layer F.Cu) (net 3))
+  (segment (start -9.778 22.074) (end -9.778 23.369) (width 0.5) (layer F.Cu) (net 3))
+  (segment (start 2.446315 33.814) (end 5.632 33.814) (width 0.5) (layer F.Cu) (net 4))
+  (segment (start -2.667 28.700685) (end 2.446315 33.814) (width 0.5) (layer F.Cu) (net 4))
+  (segment (start -2.667 28.700685) (end -2.667 28.135) (width 0.5) (layer F.Cu) (net 4))
+  (segment (start -3.430315 29.464) (end -2.667 28.700685) (width 0.5) (layer F.Cu) (net 4))
+  (segment (start -5.503685 29.464) (end -3.430315 29.464) (width 0.5) (layer F.Cu) (net 4))
+  (segment (start -6.267 28.700685) (end -5.503685 29.464) (width 0.5) (layer F.Cu) (net 4))
+  (segment (start -6.267 28.135) (end -6.267 28.700685) (width 0.5) (layer F.Cu) (net 4))
+  (segment (start -2.667 35.814) (end -2.667 35.135) (width 0.5) (layer F.Cu) (net 5))
+  (segment (start -3.302 36.449) (end -2.667 35.814) (width 0.5) (layer F.Cu) (net 5))
+  (segment (start -5.588 36.449) (end -3.302 36.449) (width 0.5) (layer F.Cu) (net 5))
+  (segment (start -6.267 35.77) (end -5.588 36.449) (width 0.5) (layer F.Cu) (net 5))
+  (segment (start -6.267 35.135) (end -6.267 35.77) (width 0.5) (layer F.Cu) (net 5))
+  (segment (start -2.667 35.700685) (end -1.918685 36.449) (width 0.5) (layer F.Cu) (net 5))
+  (segment (start -2.667 35.135) (end -2.667 35.700685) (width 0.5) (layer F.Cu) (net 5))
+  (segment (start 4.997 36.449) (end 5.632 35.814) (width 0.5) (layer F.Cu) (net 5))
+  (segment (start -1.918685 36.449) (end 4.997 36.449) (width 0.5) (layer F.Cu) (net 5))
   (zone (net 2) (net_name +3V3) (layer F.Cu) (hatch edge 0.508)
     (connect_pads yes (clearance 0.508))
@@
   )
   (zone (net 1) (net_name GND) (layer B.Cu) (hatch edge 0.508)
-    (connect_pads (clearance 0.508))
+    (connect_pads yes (clearance 0.508))
     (min_thickness 0.254)
     (fill yes (arc_segments 32) (thermal_gap 0.508) (thermal_bridge_width 0.508))

Commit message: .
Parts:
- moved SW1 9.60 mm to (0.00, 40.5), turned to 0 degrees
- moved C1 6.86 mm to (5.36, 31.8), turned to 180 degrees
- moved U1 4.47 mm to (0.00, 35.0)
- moved U2 4.47 mm to (0.00, 28.0)
Routing:
- net VBUS2: track 15.8 -> 27.6 mm
- net VBUS1: track 14.9 -> 8.71 mm
- net VBUS3: track 24.8 -> 30.4 mm
- net GND: track 1.79 -> 3.33 mm, vias 19 -> 20

Commit message: .
Parts:
- added D9: DIODE, Diode_SMD:D_SOD-323, F.Cu at (0.32, 31.6)
Routing:
- net VBUS3: track 30.4 -> 35.5 mm
- net VBUS2: track 27.6 -> 29.8 mm

Commit message: .
Parts:
- D9: footprint Diode_SMD:D_SOD-323 -> Diode_SMD:D_SMA
- moved D9 0.64 mm to (-0.32, 31.5)
Routing:
- net VBUS2: track 29.8 -> 27.6 mm
Changed lines of the file:
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@@
     (thickness 1.6)
     (drawings 15)
-    (tracks 430)
+    (tracks 429)
     (zones 0)
     (modules 15)
@@
     (add_net +3V3)
     (add_net GND)
-    (add_net "Net-(SW1-Pad1)")
-    (add_net "Net-(U1-Pad3)")
-    (add_net "Net-(U1-Pad4)")
-    (add_net "Net-(U2-Pad3)")
-    (add_net "Net-(U2-Pad4)")
     (add_net VBUS1)
     (add_net VBUS2)
     (add_net VBUS3)
   )
-  (module Diode_SMD:D_SOD-323 (layer F.Cu)
-    (at 0.3175 31.5595 180)
-    (descr SOD-323)
-    (tags SOD-323)
+  (module Diode_SMD:D_SMA (layer F.Cu)
+    (at -0.3175 31.496 180)
+    (descr "Diode SMA (DO-214AC)")
+    (tags "Diode SMA (DO-214AC)")
     (attr smd)
     (fp_text reference D9 (at 0 -1.85) (layer F.SilkS)
@@
       (effects (font (size 1 1) (thickness 0.15)))
     )
-    (fp_line (start -1.5 -0.85) (end -1.5 0.85) (layer F.SilkS) (width 0.12))
-    (fp_line (start 0.2 0) (end 0.45 0) (layer F.Fab) (width 0.1))
-    (fp_line (start 0.2 0.35) (end -0.3 0) (layer F.Fab) (width 0.1))
-    (fp_line (start 0.2 -0.35) (end 0.2 0.35) (layer F.Fab) (width 0.1))
-    (fp_line (start -0.3 0) (end 0.2 -0.35) (layer F.Fab) (width 0.1))
-    (fp_line (start -0.3 0) (end -0.5 0) (layer F.Fab) (width 0.1))
-    (fp_line (start -0.3 -0.35) (end -0.3 0.35) (layer F.Fab) (width 0.1))
-    (fp_line (start -0.9 0.7) (end -0.9 -0.7) (layer F.Fab) (width 0.1))
-    (fp_line (start 0.9 0.7) (end -0.9 0.7) (layer F.Fab) (width 0.1))
-    (fp_line (start 0.9 -0.7) (end 0.9 0.7) (layer F.Fab) (width 0.1))
-    (fp_line (start -0.9 -0.7) (end 0.9 -0.7) (layer F.Fab) (width 0.1))
-    (fp_line (start -1.6 -0.95) (end 1.6 -0.95) (layer F.CrtYd) (width 0.05))
-    (fp_line (start 1.6 -0.95) (end 1.6 0.95) (layer F.CrtYd) (width 0.05))
-    (fp_line (start -1.6 0.95) (end 1.6 0.95) (layer F.CrtYd) (width 0.05))
-    (fp_line (start -1.6 -0.95) (end -1.6 0.95) (layer F.CrtYd) (width 0.05))
-    (fp_line (start -1.5 0.85) (end 1.05 0.85) (layer F.SilkS) (width 0.12))
-    (fp_line (start -1.5 -0.85) (end 1.05 -0.85) (layer F.SilkS) (width 0.12))
-    (pad 2 smd rect (at 1.05 0 180) (size 0.6 0.45) (layers F.Cu F.Paste F.Mask)
+    (fp_line (start -3.4 -1.65) (end -3.4 1.65) (layer F.SilkS) (width 0.12))
+    (fp_line (start 2.3 1.5) (end -2.3 1.5) (layer F.Fab) (width 0.1))
+    (fp_line (start -2.3 1.5) (end -2.3 -1.5) (layer F.Fab) (width 0.1))
+    (fp_line (start 2.3 -1.5) (end 2.3 1.5) (layer F.Fab) (width 0.1))
+    (fp_line (start 2.3 -1.5) (end -2.3 -1.5) (layer F.Fab) (width 0.1))
+    (fp_line (start -3.5 -1.75) (end 3.5 -1.75) (layer F.CrtYd) (width 0.05))
+    (fp_line (start 3.5 -1.75) (end 3.5 1.75) (layer F.CrtYd) (width 0.05))
+    (fp_line (start 3.5 1.75) (end -3.5 1.75) (layer F.CrtYd) (width 0.05))
+    (fp_line (start -3.5 1.75) (end -3.5 -1.75) (layer F.CrtYd) (width 0.05))
+    (fp_line (start -0.64944 0.00102) (end -1.55114 0.00102) (layer F.Fab) (width 0.1))
+    (fp_line (start 0.50118 0.00102) (end 1.4994 0.00102) (layer F.Fab) (width 0.1))
+    (fp_line (start -0.64944 -0.79908) (end -0.64944 0.80112) (layer F.Fab) (width 0.1))
+    (fp_line (start 0.50118 0.75032) (end 0.50118 -0.79908) (layer F.Fab) (width 0.1))
+    (fp_line (start -0.64944 0.00102) (end 0.50118 0.75032) (layer F.Fab) (width 0.1))
+    (fp_line (start -0.64944 0.00102) (end 0.50118 -0.79908) (layer F.Fab) (width 0.1))
+    (fp_line (start -3.4 1.65) (end 2 1.65) (layer F.SilkS) (width 0.12))
+    (fp_line (start -3.4 -1.65) (end 2 -1.65) (layer F.SilkS) (width 0.12))
+    (pad 2 smd rect (at 2 0 180) (size 2.5 1.8) (layers F.Cu F.Paste F.Mask)
       (net 4 VBUS2))
-    (pad 1 smd rect (at -1.05 0 180) (size 0.6 0.45) (layers F.Cu F.Paste F.Mask)
+    (pad 1 smd rect (at -2 0 180) (size 2.5 1.8) (layers F.Cu F.Paste F.Mask)
       (net 3 VBUS3))
-    (model ${KISYS3DMOD}/Diode_SMD.3dshapes/D_SOD-323.wrl
+    (model ${KISYS3DMOD}/Diode_SMD.3dshapes/D_SMA.wrl
       (at (xyz 0 0 0))
       (scale (xyz 1 1 1))
@@
   (segment (start -9.424446 23.595553) (end -8.481553 24.538446) (width 0.5) (layer F.Cu) (net 3))
   (segment (start 1.3675 31.5595) (end 1.905 31.5595) (width 0.5) (layer F.Cu) (net 3))
-  (segment (start 1.905 31.5595) (end 3.2385 30.226) (width 0.5) (layer F.Cu) (net 3))
   (segment (start 5.842 30.226) (end 5.842 36.33) (width 0.5) (layer F.Cu) (net 3))
+  (segment (start 5.842 26.916) (end 5.842 30.226) (width 0.5) (layer F.Cu) (net 3))
+  (segment (start 1.6825 31.496) (end 1.9685 31.496) (width 0.5) (layer F.Cu) (net 3))
   (segment (start 3.2385 30.226) (end 5.842 30.226) (width 0.5) (layer F.Cu) (net 3))
-  (segment (start 5.842 26.916) (end 5.842 30.226) (width 0.5) (layer F.Cu) (net 3))
+  (segment (start 1.9685 31.496) (end 3.2385 30.226) (width 0.5) (layer F.Cu) (net 3))
   (segment (start 2 37.75) (end 2 38.386) (width 0.5) (layer F.Cu) (net 4))
   (segment (start 0.516 39.37) (end 0.575229 39.368545) (width 0.5) (layer F.Cu) (net 4))
@@
   (segment (start -1.612379 27.382927) (end -1.587867 27.357182) (width 0.5) (layer F.Cu) (net 4))
   (segment (start -1.587867 27.357182) (end -1.366817 27.136132) (width 0.5) (layer F.Cu) (net 4))
-  (segment (start -0.7325 31.5595) (end -1.4605 31.5595) (width 0.5) (layer F.Cu) (net 4))
-  (segment (start -1.4605 31.5595) (end -2.54 30.48) (width 0.5) (layer F.Cu) (net 4))
   (segment (start -2.54 30.48) (end -2.948446 30.888446) (width 0.5) (layer F.Cu) (net 4))
   (segment (start -2.153553 30.093553) (end -2.54 30.48) (width 0.5) (layer F.Cu) (net 4))
