File: led-ring.sch (KiCad schematic (older format))
At the start: 14 parts, among them SW1 DP3T, U1 USB-C-6-PIN, U2 USB-C-6-PIN, U3 AMS1117-3.3

Commit message: .
Parts:
- added D?: DIODE, Diode_SMD:D_SOD-323, symbol pspice:DIODE
Connections:
- net VBUS2: now also D?.2 (A)
- net VBUS3: now also D?.1 (K)
Changed lines of the file:
@@
 Wire Wire Line
 	4000 1400 4050 1400
+Text GLabel 5650 2350 0    50   Input ~ 0
+VBUS3
+Text GLabel 6450 2350 2    50   Input ~ 0
+VBUS2
+$Comp
+L pspice:DIODE D?
+U 1 1 617034F7
+P 6050 2350
+F 0 "D?" H 6050 2615 50  0000 C CNN
+F 1 "DIODE" H 6050 2524 50  0000 C CNN
+F 2 "Diode_SMD:D_SOD-323" H 6050 2350 50  0001 C CNN
+F 3 "~" H 6050 2350 50  0001 C CNN
+	1    6050 2350
+	1    0    0    -1
+$EndComp
+Wire Wire Line
+	5650 2350 5850 2350
+Wire Wire Line
+	6250 2350 6450 2350
 $EndSCHEMATC

Commit message: .
Parts:
- D9: renamed from D?; footprint Diode_SMD:D_SOD-323 -> Diode_SMD:D_SMA
Changed lines of the file:
@@
 VBUS2
 $Comp
-L pspice:DIODE D?
+L pspice:DIODE D9
 U 1 1 617034F7
 P 6050 2350
-F 0 "D?" H 6050 2615 50  0000 C CNN
+F 0 "D9" H 6050 2615 50  0000 C CNN
 F 1 "DIODE" H 6050 2524 50  0000 C CNN
-F 2 "Diode_SMD:D_SOD-323" H 6050 2350 50  0001 C CNN
+F 2 "Diode_SMD:D_SMA" H 6050 2350 50  0001 C CNN
 F 3 "~" H 6050 2350 50  0001 C CNN
 	1    6050 2350
